Commit message: update bimanual tele

File: src/simulation/mani_skill/assets/robots/openarm_bi/openarm_bi.urdf (robot description, URDF)
Before this commit: robot openarm, 26 links, 25 joints
Links:
- link openarm_body_link0: geometry collision mesh filename=meshes/body/v10/collision/body_link0_symp.stl scale=0.001 0.001 0.001; visual mesh filename=meshes/body/v10/visual/body_link0.dae scale=0.001 0.001 0.001
- link openarm_left_hand: geometry collision mesh filename=meshes/ee/openarm_hand/collision/hand.stl scale=0.001 0.001 0.001; visual mesh filename=meshes/ee/openarm_hand/visual/hand.dae scale=0.001 0.001 0.001
- link openarm_left_left_finger: geometry collision mesh filename=meshes/ee/openarm_hand/collision/finger.stl scale=0.001 0.001 0.001; visual mesh filename=meshes/ee/openarm_hand/visual/finger.dae scale=0.001 0.001 0.001
- link openarm_left_link0: geometry collision mesh filename=meshes/arm/v10/collision/link0_symp.stl scale=0.001 -0.001 0.001; visual mesh filename=meshes/arm/v10/visual/link0.dae scale=0.001 -0.001 0.001
- link openarm_left_link1: geometry collision mesh filename=meshes/arm/v10/collision/link1_symp.stl scale=0.001 -0.001 0.001; visual mesh filename=meshes/arm/v10/visual/link1.dae scale=0.001 -0.001 0.001
- link openarm_left_link2: geometry collision mesh filename=meshes/arm/v10/collision/link2_symp.stl scale=0.001 -0.001 0.001; visual mesh filename=meshes/arm/v10/visual/link2.dae scale=0.001 -0.001 0.001
- link openarm_left_link3: geometry collision mesh filename=meshes/arm/v10/collision/link3_symp.stl scale=0.001 -0.001 0.001; visual mesh filename=meshes/arm/v10/visual/link3.dae scale=0.001 -0.001 0.001
- link openarm_left_link4: geometry collision mesh filename=meshes/arm/v10/collision/link4_symp.stl scale=0.001 0.001 0.001; visual mesh filename=meshes/arm/v10/visual/link4.dae scale=0.001 0.001 0.001
- link openarm_left_link5: geometry collision mesh filename=meshes/arm/v10/collision/link5_symp.stl scale=0.001 -0.001 0.001; visual mesh filename=meshes/arm/v10/visual/link5.dae scale=0.001 -0.001 0.001
- link openarm_left_link6: geometry collision mesh filename=meshes/arm/v10/collision/link6_symp.stl scale=0.001 -0.001 0.001; visual mesh filename=meshes/arm/v10/visual/link6.dae scale=0.001 -0.001 0.001
- link openarm_left_link7: geometry collision mesh filename=meshes/arm/v10/collision/link7_symp.stl scale=0.001 -0.001 0.001; visual mesh filename=meshes/arm/v10/visual/link7.dae scale=0.001 -0.001 0.001
- link openarm_left_right_finger: geometry collision mesh filename=meshes/ee/openarm_hand/collision/finger.stl scale=0.001 -0.001 0.001; visual mesh filename=meshes/ee/openarm_hand/visual/finger.dae scale=0.001 -0.001 0.001
- link openarm_right_hand: geometry collision mesh filename=meshes/ee/openarm_hand/collision/hand.stl scale=0.001 0.001 0.001; visual mesh filename=meshes/ee/openarm_hand/visual/hand.dae scale=0.001 0.001 0.001
- link openarm_right_left_finger: geometry collision mesh filename=meshes/ee/openarm_hand/collision/finger.stl scale=0.001 0.001 0.001; visual mesh filename=meshes/ee/openarm_hand/visual/finger.dae scale=0.001 0.001 0.001
- link openarm_right_link0: geometry collision mesh filename=meshes/arm/v10/collision/link0_symp.stl scale=0.001 0.001 0.001; visual mesh filename=meshes/arm/v10/visual/link0.dae scale=0.001 0.001 0.001
- link openarm_right_link1: geometry collision mesh filename=meshes/arm/v10/collision/link1_symp.stl scale=0.001 0.001 0.001; visual mesh filename=meshes/arm/v10/visual/link1.dae scale=0.001 0.001 0.001
- link openarm_right_link2: geometry collision mesh filename=meshes/arm/v10/collision/link2_symp.stl scale=0.001 0.001 0.001; visual mesh filename=meshes/arm/v10/visual/link2.dae scale=0.001 0.001 0.001
- link openarm_right_link3: geometry collision mesh filename=meshes/arm/v10/collision/link3_symp.stl scale=0.001 0.001 0.001; visual mesh filename=meshes/arm/v10/visual/link3.dae scale=0.001 0.001 0.001
- link openarm_right_link4: geometry collision mesh filename=meshes/arm/v10/collision/link4_symp.stl scale=0.001 0.001 0.001; visual mesh filename=meshes/arm/v10/visual/link4.dae scale=0.001 0.001 0.001
- link openarm_right_link5: geometry collision mesh filename=meshes/arm/v10/collision/link5_symp.stl scale=0.001 0.001 0.001; visual mesh filename=meshes/arm/v10/visual/link5.dae scale=0.001 0.001 0.001
- link openarm_right_link6: geometry collision mesh filename=meshes/arm/v10/collision/link6_symp.stl scale=0.001 0.001 0.001; visual mesh filename=meshes/arm/v10/visual/link6.dae scale=0.001 0.001 0.001
- link openarm_right_link7: geometry collision mesh filename=meshes/arm/v10/collision/link7_symp.stl scale=0.001 0.001 0.001; visual mesh filename=meshes/arm/v10/visual/link7.dae scale=0.001 0.001 0.001
- link openarm_right_right_finger: geometry collision mesh filename=meshes/ee/openarm_hand/collision/finger.stl scale=0.001 -0.001 0.001; visual mesh filename=meshes/ee/openarm_hand/visual/finger.dae scale=0.001 -0.001 0.001
